File: hardware/SN74HC165 Shift-In Breakout-v11.brd (EAGLE design)
At the start: 20.3 x 30.5 mm, 10 parts, among them U1 74HC165D

Commit message: Fixed v11 BRD file
Parts:
- moved JP2 27.9 mm to (5.08, 29.2)
- moved JP3 27.9 mm to (5.08, 1.27)
Routing:
- net SERIAL_OUT: track 20.9 -> 12.0 mm, vias 1 -> 0
- net SERIAL_IN: track 13.8 -> 20.7 mm, vias 0 -> 1
Other:
- board text added: "v11"
- board text removed: "v10\"
Changed lines of the file:
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@@
 <text x="15.24" y="-17.78" size="1.778" layer="49" font="vector" ratio="15">Jordan McConnell</text>
 <text x="9.398" y="24.003" size="1.27" layer="22" font="vector" ratio="15" rot="MR270">74HC165 Shift-In</text>
-<text x="2.159" y="29.718" size="1.27" layer="16" font="vector" ratio="15" rot="MR270">v10\</text>
+<text x="2.159" y="29.718" size="1.27" layer="16" font="vector" ratio="15" rot="MR270">v11</text>
 </plain>
 <attributes>
@@
 <element name="U1" library="SparkFun-DigitalIC" package="SO16" value="74HC165D" x="11.43" y="15.24" rot="R270"/>
 <element name="JP1" library="SparkFun-Connectors" package="1X08" value="" x="1.27" y="24.13" rot="R270"/>
-<element name="JP2" library="SparkFun-Connectors" package="1X06" value="" x="5.08" y="1.27"/>
-<element name="JP3" library="SparkFun-Connectors" package="1X06" value="" x="5.08" y="29.21"/>
+<element name="JP2" library="SparkFun-Connectors" package="1X06" value="" x="5.08" y="29.21"/>
+<element name="JP3" library="SparkFun-Connectors" package="1X06" value="" x="5.08" y="1.27"/>
 <element name="C1" library="SparkFun-Passives" package="0402-CAP" value=".1uF" x="7.62" y="8.89" rot="R180"/>
 <element name="JP4" library="SparkFun-Aesthetics" package="SFE-LOGO-FLAME" value="LOGO-SFESK" x="16.51" y="16.129" rot="R270"/>
@@
 <wire x1="11.557" y1="26.67" x2="6.35" y2="26.67" width="0.254" layer="1"/>
 <wire x1="6.35" y1="26.67" x2="5.08" y2="27.94" width="0.254" layer="1"/>
-<wire x1="5.08" y1="27.94" x2="5.08" y2="29.21" width="0.254" layer="1"/>
 <via x="5.08" y="8.89" extent="1-16" drill="0.508"/>
 <wire x1="5.08" y1="1.27" x2="5.08" y2="8.89" width="1.016" layer="1"/>
@@
 <wire x1="10.16" y1="15.24" x2="10.16" y2="8.89" width="0.254" layer="16"/>
 <wire x1="10.16" y1="15.24" x2="11.43" y2="16.51" width="0.254" layer="16"/>
+<wire x1="5.08" y1="27.94" x2="5.08" y2="29.21" width="0.254" layer="1"/>
 </signal>
 <signal name="GND">
@@
 <via x="12.319" y="12.446" extent="1-16" drill="0.508"/>
 <wire x1="12.192" y1="5.588" x2="15.24" y2="2.54" width="0.254" layer="1"/>
-<wire x1="15.24" y1="2.54" x2="15.24" y2="1.27" width="0.254" layer="1"/>
 <wire x1="12.192" y1="5.588" x2="12.192" y2="12.319" width="0.254" layer="1"/>
 <wire x1="12.192" y1="12.319" x2="12.319" y2="12.446" width="0.254" layer="1"/>
@@
 <via x="13.716" y="24.384" extent="1-16" drill="0.508"/>
 <wire x1="13.716" y1="24.384" x2="14.224" y2="24.384" width="0.254" layer="16"/>
+<wire x1="15.24" y1="2.54" x2="15.24" y2="1.27" width="0.254" layer="1"/>
 </signal>
 <signal name="CLK">
@@
 <contactref element="U1" pad="10"/>
 <contactref element="JP2" pad="6"/>
-<wire x1="14.23" y1="12.065" x2="13.462" y2="12.065" width="0.254" layer="1"/>
-<wire x1="13.462" y1="12.065" x2="12.954" y2="11.557" width="0.254" layer="1"/>
-<wire x1="12.954" y1="11.557" x2="12.954" y2="6.096" width="0.254" layer="1"/>
-<wire x1="12.954" y1="6.096" x2="17.78" y2="1.27" width="0.254" layer="1"/>
+<wire x1="14.23" y1="12.065" x2="17.78" y2="12.065" width="0.254" layer="1"/>
+<via x="17.78" y="12.065" extent="1-16" drill="0.508"/>
+<wire x1="17.78" y1="12.065" x2="17.78" y2="29.21" width="0.254" layer="16"/>
 </signal>
 <signal name="SERIAL_OUT">
 <contactref element="U1" pad="9"/>
 <contactref element="JP3" pad="6"/>
-<wire x1="14.23" y1="10.795" x2="16.002" y2="10.795" width="0.254" layer="1"/>
-<via x="16.002" y="10.795" extent="1-16" drill="0.508"/>
-<wire x1="16.002" y1="10.795" x2="16.002" y2="10.922" width="0.254" layer="16"/>
-<wire x1="16.002" y1="10.922" x2="17.78" y2="12.7" width="0.254" layer="16"/>
-<wire x1="17.78" y1="12.7" x2="17.78" y2="29.21" width="0.254" layer="16"/>
+<wire x1="14.23" y1="10.795" x2="15.875" y2="10.795" width="0.254" layer="1"/>
+<wire x1="15.875" y1="10.795" x2="16.51" y2="10.16" width="0.254" layer="1"/>
+<wire x1="16.51" y1="10.16" x2="16.51" y2="2.54" width="0.254" layer="1"/>
+<wire x1="16.51" y1="2.54" x2="17.78" y2="1.27" width="0.254" layer="1"/>
 </signal>
 </signals>
